File: SBSP Control Board/SBSP Control Board.kicad_sch (KiCad schematic)
At the start: 18 parts, among them J1 Conn_02x08_Odd_Even, U1 ADAR1000ACCZN

Commit message: started working on level shifting
Parts:
- added C10: 100pF, symbol Device:C
- added C11, C13: 1uf, symbol Device:C
- added C12, C14: TBD, symbol Device:C
- added C8: 4.7pF, symbol Device:C
- added C9: 0.01uF, symbol Device:C
- added R10, R11: 10k, symbol Device:R
Connections:
- net AVDD1 is gone; now on net GND: U1.B11 (AVDD)
- net AVDD3: now also C10.1, C8.1, C9.1
- net CREG3: now also C11.1, C12.1
- net CREG4: now also C13.1, C14.1
- net GND: now also C10.2, C11.2, C12.2, C13.2, C14.2, C8.2, C9.2, R10.1, R11.1
- net ADDR0: no longer names the net of U1.N4 (ADDR0)
- net ADDR0: now also R11.2
- net ADDR1: no longer names the net of U1.N5 (ADDR1)
- net ADDR1: now also R10.2
Other:
- added sheet TX1 (TX1.kicad_sch)
- added sheet TX2 (TX1.kicad_sch)
- added sheet TX4 (TX1.kicad_sch)
- moved on the sheet: U1C
