File: SBSP Control Board/SBSP Control Board.kicad_sch (KiCad schematic)
At the start: 27 parts, among them J1 Conn_02x08_Odd_Even, U1 ADAR1000ACCZN

Commit message: finished first sch rev. started layout
need to add some more things but this is for a basic demo and to get an understanding of the length of the traces needed.
Parts:
- removed C1: 4.7pf, symbol Device:C
- removed C10: 100pF, symbol Device:C
- removed C2: 0.01uf, symbol Device:C
- removed C3: 100pf, symbol Device:C
- removed C8: 4.7pF, symbol Device:C
- removed C9: 0.01uF, symbol Device:C
- removed R1: 75, symbol Device:R
- added C59: 100pF, Capacitor_SMD:C_1206_3216Metric, symbol Device:C
- added C60: 0.01uF, Capacitor_SMD:C_1206_3216Metric, symbol Device:C
- added C61: 4.7pF, Capacitor_SMD:C_1206_3216Metric, symbol Device:C
- added J10, J11, J12, J13, J14, J15, J16, J17, J2, J3, J4, J5, J6, J7, J8, J9: Conn_Coaxial, Connector_Coaxial:SMA_Amphenol_132289_EdgeMount, symbol Connector:Conn_Coaxial
- added J18, J19: Conn_01x02_Socket, Connector_PinSocket_2.54mm:PinSocket_1x02_P2.54mm_Vertical_SMD_Pin1Left, symbol Connector:Conn_01x02_Socket
- added R12: 10k, Resistor_SMD:R_1206_3216Metric, symbol Device:R
- C11, C12, C13, C14, C4, C5, C6, C7: footprint (none) -> Capacitor_SMD:C_1206_3216Metric
- R10, R11, R2, R3, R4, R5, R6, R7, R8, R9: footprint (none) -> Resistor_SMD:R_1206_3216Metric
Connections:
- net CSB: no longer U1.M3 (CSB)
- net GND: now also C59.2, C60.2, C61.2, J10.2 (Ext), J11.2 (Ext), J12.2 (Ext), J13.2 (Ext), J14.2 (Ext), J15.2 (Ext), J16.2 (Ext), J17.2 (Ext), J18.2 (Pin_2), J19.2 (Pin_2), J2.2 (Ext), J3.2 (Ext), J4.2 (Ext), J5.2 (Ext), J6.2 (Ext), J7.2 (Ext), J8.2 (Ext), J9.2 (Ext), R12.1
- net RX_LOAD: no longer U1.N2 (RX_LOAD)
- net SCLK: no longer U1.M6 (SCLK)
- net SDIO: no longer U1.M5 (SDIO)
- net SDO: no longer U1.M4 (SDO)
- net TR: no longer U1.N6 (TR)
- net TX_LOAD: no longer U1.N3 (TX_LOAD)
- net AVDD3 renamed +3.3V
- net +3.3V: now also C59.1, C60.1, C61.1, J18.1 (Pin_1)
- net LNA_B1: no longer names the net of U1.A11 (LNA_BIAS)
- net PA_B1: no longer names the net of U1.A10 (PA_BIAS1)
- net PA_B2: no longer names the net of U1.A9 (PA_BIAS2)
- net PA_B3: no longer names the net of U1.A5 (PA_BIAS3)
- net PA_B4: no longer names the net of U1.A4 (PA_BIAS4)
- net PA_ON: no longer names the net of U1.B3 (PA_ON)
- net RF_IO renamed PLL_IN
- net RX1: no longer names the net of U1.J13 (RX1)
- net RX2: no longer names the net of U1.C13 (RX2)
- net RX3: no longer names the net of U1.E1 (RX3)
- net RX4: no longer names the net of U1.L1 (RX4)
- net TR_POL: no longer names the net of U1.B4 (TR_POL)
- net TR_SW_NEG: no longer names the net of U1.A3 (TR_SW_NEG)
- new net: R12.2, U1.N2 (RX_LOAD)
- new net +1.8V: J19.1 (Pin_1)
- new net ADAR_CS_STAGE1_1V8: U1.M3 (CSB)
- new net ADAR_SCLK_1V8: U1.M6 (SCLK)
- new net ADAR_SDIO_1V8: U1.M5 (SDIO)
- new net ADAR_SDO_STAGE1_1V8: U1.M4 (SDO)
- new net ADAR_TR_1V8: U1.N6 (TR)
- new net ADAR_TX_LOAD_1V8: U1.N3 (TX_LOAD)
- new net OUT1: J2.1 (In)
- new net OUT10: J11.1 (In)
- new net OUT11: J12.1 (In)
- new net OUT12: J13.1 (In)
- new net OUT13: J14.1 (In)
- new net OUT14: J15.1 (In)
- new net OUT15: J16.1 (In)
- new net OUT16: J17.1 (In)
- new net OUT2: J3.1 (In)
- new net OUT3: J4.1 (In)
- new net OUT4: J5.1 (In)
- new net OUT5: J6.1 (In)
- new net OUT6: J7.1 (In)
- new net OUT7: J8.1 (In)
- new net OUT8: J9.1 (In)
- new net OUT9: J10.1 (In)
- no-connect marks 0 -> 13
Other:
- added sheet TX3 (TX3.kicad_sch)
- sheet TX2: file TX1.kicad_sch -> TX2.kicad_sch
- sheet TX4: file TX1.kicad_sch -> TX4.kicad_sch
- note added: "PU/PD"
- note added: "TODO: 1. are we having an onboard MCU for this? or are we just setting the control and forgetting about it 2. are we using the det detection pins? 3. add a level shifter for the 1.8v logic"
- note added: "WILL NEED A LEVEL TRANSISTOR!!! 3.3V ->1.8V"
- moved on the sheet: C11, C12, C13, C14, C4, C5, C6, C7, U1B
