File: SBSP Control Board/SBSP Control Board.kicad_sch (KiCad schematic)
At the start: 50 parts, among them J10 Conn_Coaxial, J11 Conn_Coaxial, J12 Conn_Coaxial, J13 Conn_Coaxial, J14 Conn_Coaxial, J15 Conn_Coaxial, J16 Conn_Coaxial, J17 Conn_Coaxial, J18 Conn_01x02_Socket, J19 Conn_01x02_Socket, J2 Conn_Coaxial, J20 Conn_01x20_Socket, J21 Conn_01x20_Socket, J3 Conn_Coaxial, J4 Conn_Coaxial, J5 Conn_Coaxial, J6 Conn_Coaxial, J7 Conn_Coaxial, J8 Conn_Coaxial, J9 Conn_Coaxial, U1 ADAR1000ACCZN, U5 SN74AVC4T245PW

Commit message: finished implementing level shifting
just need to go look and do a run through to make sure it's all okay. also need to look into the power requirements for the +3/-5/-3 and make sure the nets are all correct. just double check the pdf with what we have wired.
Parts:
- removed J10, J11, J12, J13, J14, J15, J16, J17, J9: Conn_Coaxial, Connector_Coaxial:SMA_Amphenol_132289_EdgeMount, symbol Connector:Conn_Coaxial
Other:
- removed sheet TX2
- removed sheet TX3
- removed sheet TX4
