File: SBSP Control Board/SBSP Control Board.kicad_pcb (KiCad board)
At the start: 4 copper layers, 201.7 x 75.1 mm, 93 parts, among them J10 Conn_Coaxial, J11 Conn_Coaxial, J12 Conn_Coaxial, J13 Conn_Coaxial, J14 Conn_Coaxial, J15 Conn_Coaxial, J16 Conn_Coaxial, J17 Conn_Coaxial, J18 Conn_01x02_Socket, J19 Conn_01x02_Socket, J2 Conn_Coaxial, J3 Conn_Coaxial, J4 Conn_Coaxial, J5 Conn_Coaxial, J6 Conn_Coaxial, J7 Conn_Coaxial, J8 Conn_Coaxial, J9 Conn_Coaxial, U1 ADAR1000ACCZN, U2 ADAR1000ACCZN, U3 ADAR1000ACCZN, U4 ADAR1000ACCZN, U6 ADAR1000ACCZN

Commit message: first rev of trans. line routed
Parts:
- moved U4 170.8 mm to (161.3, 56.0), turned to 180 degrees
- moved U1 169.1 mm to (135.9, 69.4), turned to 180 degrees
- moved U3 123.6 mm to (110.6, 56.0), turned to 180 degrees
- moved U2 79.6 mm to (60.0, 56.0), turned to 180 degrees
- moved J6 12.8 mm to (104.2, 33.4)
- moved J8 12.8 mm to (129.6, 33.4)
- moved J12 12.7 mm to (180.3, 33.3)
- moved J13 12.7 mm to (167.6, 33.3)
- moved J14 12.7 mm to (205.7, 33.3)
- moved J15 12.7 mm to (193.0, 33.3)
- moved J2 12.7 mm to (53.3, 33.3)
- moved J3 12.7 mm to (40.6, 33.3)
- moved J7 12.7 mm to (91.4, 33.3)
- moved J10 12.7 mm to (154.9, 33.3)
- moved J11 12.7 mm to (142.2, 33.3)
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Connections:
- U2 pad A7: TX1 -> TX2
- U3 pad A7: TX2 -> TX1
- U4 pad A7: TX3 -> TX4
- U6 pad A7: TX4 -> TX3
Routing:
- net TX3: track 0.00 -> 78.5 mm
- net TX2: track 0.00 -> 78.5 mm
- net TX4: track 0.00 -> 77.7 mm
- net TX1: track 0.00 -> 77.7 mm
- net OUT15: track 0.00 -> 32.5 mm
- net OUT14: track 0.00 -> 32.5 mm
- net OUT11: track 0.00 -> 32.5 mm
- net OUT7: track 0.00 -> 32.5 mm
- net OUT3: track 0.00 -> 32.5 mm
- net OUT2: track 0.00 -> 32.4 mm
- net OUT6: track 0.00 -> 32.4 mm
- net OUT10: track 0.00 -> 32.4 mm
- net OUT16: track 0.00 -> 32.2 mm
- net OUT12: track 0.00 -> 32.2 mm
- net OUT8: track 0.00 -> 32.2 mm
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- added copper zone on F.Cu, net GND
Other:
- board size 201.7 x 75.1 mm -> 201.7 x 63.5 mm

Commit message: 'finished' the first IC routing
need to re do and see what connections we need to make for programming. also need to see about better ground connections to the IC.
Parts:
- removed C12, C14, C5, C7: TBD, Capacitor_SMD:C_1206_3216Metric
- added J1: Conn_02x08_Odd_Even, Resistor_SMD:R_0603_1608Metric, F.Cu at (1.50, 0.76)
- C11, C13, C4, C59, C6, C60, C61: footprint Capacitor_SMD:C_1206_3216Metric -> Resistor_SMD:R_0603_1608Metric; moved to B.Cu
- C15, C16, C17, C18, C19, C20, C21, C22, C23, C24, C25, C26, C27, C28, C29, C30, C31, C32, C33, C34, C35, C36, C37, C38, C39, C40, C41, C42, C43, C44, C45, C46, C47, C48, C49, C50, C51, C52, C53, C54, C55, C56, C57, C58: footprint Capacitor_SMD:C_1206_3216Metric -> Resistor_SMD:R_0603_1608Metric
- R1, R13, R14, R15, R2, R3, R4, R5, R6, R7, R8, R9: footprint Resistor_SMD:R_1206_3216Metric -> Resistor_SMD:R_0603_1608Metric
- R10, R11, R12: footprint Resistor_SMD:R_1206_3216Metric -> Resistor_SMD:R_0603_1608Metric; moved to B.Cu
- moved C4 217.9 mm to (135.4, 69.1), turned to -90 degrees
- moved C6 214.1 mm to (133.8, 69.1), turned to -90 degrees
- moved C13 211.3 mm to (136.2, 63.4), turned to 90 degrees
- moved C11 211.2 mm to (134.6, 63.7), turned to 90 degrees
- moved R10 209.4 mm to (142.0, 62.1), turned to 180 degrees
- moved R11 209.1 mm to (142.0, 63.7), turned to 180 degrees
- moved R12 208.7 mm to (142.0, 65.2), turned to 180 degrees
- moved C59 204.8 mm to (132.3, 61.3), turned to 180 degrees
- moved C60 204.3 mm to (132.3, 62.9), turned to 180 degrees
- moved C61 203.8 mm to (132.3, 64.5), turned to 180 degrees
Routing:
- net GND: track 0.00 -> 89.1 mm, vias 1117 -> 1044
- net Net-(U1A-ADDR1): track 0.00 -> 6.72 mm, vias 0 -> 1
- net +3.3V: track 0.00 -> 6.47 mm, vias 0 -> 2
- net Net-(U1A-ADDR0): track 0.00 -> 5.55 mm, vias 0 -> 1
- net Net-(U1A-RX_LOAD): track 0.00 -> 3.68 mm, vias 0 -> 1
- net /CREG4: track 0.00 -> 2.76 mm, vias 0 -> 1
- net /CREG2: track 0.00 -> 2.21 mm, vias 0 -> 1
- net /CREG3: track 0.00 -> 1.95 mm, vias 0 -> 1
- net /CREG1: track 0.00 -> 1.40 mm, vias 0 -> 1

Commit message: finished passive layout for IC's
Parts:
- removed C15, C17, C19, C21, C24, C26, C28, C30, C32, C34, C36, C38, C40, C42, C44, C46: TBD, Resistor_SMD:R_0603_1608Metric
- C16, C18, C20, C22, C23, C25, C27, C29, C31, C33, C35, C37, C39, C41, C43, C45, C47, C48, C49, C50, C51, C52, C53, C54, C55, C56, C57, C58, R1, R13, R14, R15: moved to B.Cu
- moved C39 267.9 mm to (212.9, 54.8)
- moved C41 263.9 mm to (209.8, 54.7), turned to 180 degrees
- moved C43 263.0 mm to (210.0, 50.5), turned to 90 degrees
- moved C45 260.4 mm to (211.6, 50.5), turned to 90 degrees
- moved R15 257.8 mm to (214.5, 50.6), turned to -90 degrees
- moved C56 255.5 mm to (207.7, 48.3), turned to 180 degrees
- moved C57 255.3 mm to (207.7, 49.8), turned to 180 degrees
- moved C58 255.1 mm to (207.7, 51.4), turned to 180 degrees
- moved C31 214.8 mm to (162.1, 54.8)
- moved C35 211.7 mm to (159.7, 50.3), turned to 90 degrees
- moved C33 211.3 mm to (158.9, 54.8), turned to 180 degrees
- moved C37 208.0 mm to (161.2, 50.3), turned to 90 degrees
- moved R14 205.0 mm to (163.8, 50.5), turned to -90 degrees
- moved C53 203.7 mm to (157.3, 48.0), turned to 180 degrees
- moved C54 203.6 mm to (157.3, 49.5), turned to 180 degrees
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Connections:
- U4 pad M10: unconnected-(U4B-AVDD3-PadM10) -> +3.3V
- U4 pad N11: unconnected-(U4B-AVDD3-PadN11) -> +3.3V
Routing:
- net +3.3V: track 6.47 -> 32.3 mm, vias 2 -> 5
- net Net-(U4B-CREG4): track 0.00 -> 2.67 mm, vias 0 -> 1
- net Net-(U2B-CREG3): track 0.00 -> 2.24 mm, vias 0 -> 1
- net Net-(U6B-CREG4): track 0.00 -> 2.14 mm, vias 0 -> 1
- net Net-(U6B-CREG3): track 0.00 -> 2.13 mm, vias 0 -> 1
- net Net-(U3B-CREG4): track 0.00 -> 2.13 mm, vias 0 -> 1
- net Net-(U2B-CREG4): track 0.00 -> 1.98 mm, vias 0 -> 1
- net Net-(U4B-CREG3): track 0.00 -> 1.91 mm, vias 0 -> 1
- net Net-(U3B-CREG1): track 0.00 -> 1.90 mm, vias 0 -> 1
- net Net-(U3A-RX_LOAD): track 0.00 -> 1.70 mm, vias 0 -> 1
- net Net-(U2B-CREG1): track 0.00 -> 1.70 mm, vias 0 -> 1
- net Net-(U2A-RX_LOAD): track 0.00 -> 1.64 mm, vias 0 -> 1
- net Net-(U4A-RX_LOAD): track 0.00 -> 1.63 mm, vias 0 -> 1
- net Net-(U6A-RX_LOAD): track 0.00 -> 1.60 mm, vias 0 -> 1
- net Net-(U3B-CREG3): track 0.00 -> 1.56 mm, vias 0 -> 1
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- added copper zone on B.Cu, net GND
