File: SBSP Control Board/SBSP Control Board.kicad_pcb (KiCad board)
At the start: 4 copper layers, 201.7 x 63.5 mm, 74 parts, among them J1 Conn_02x08_Odd_Even, J10 Conn_Coaxial, J11 Conn_Coaxial, J12 Conn_Coaxial, J13 Conn_Coaxial, J14 Conn_Coaxial, J15 Conn_Coaxial, J16 Conn_Coaxial, J17 Conn_Coaxial, J18 Conn_01x02_Socket, J19 Conn_01x02_Socket, J2 Conn_Coaxial, J3 Conn_Coaxial, J4 Conn_Coaxial, J5 Conn_Coaxial, J6 Conn_Coaxial, J7 Conn_Coaxial, J8 Conn_Coaxial, J9 Conn_Coaxial, U1 ADAR1000ACCZN, U2 ADAR1000ACCZN, U3 ADAR1000ACCZN, U4 ADAR1000ACCZN, U6 ADAR1000ACCZN

Commit message: finished implementing level shifting
just need to go look and do a run through to make sure it's all okay. also need to look into the power requirements for the +3/-5/-3 and make sure the nets are all correct. just double check the pdf with what we have wired.
Parts:
- removed C23, C25, C27, C29, C31, C33, C35, C37, C39, C41, C43, C45: 1uf, Resistor_SMD:R_0603_1608Metric
- removed C50, C53, C56: 100pF, Resistor_SMD:R_0603_1608Metric
- removed C51, C54, C57: 0.01uF, Resistor_SMD:R_0603_1608Metric
- removed C52, C55, C58: 4.7pF, Resistor_SMD:R_0603_1608Metric
- removed J1: Conn_02x08_Odd_Even, Resistor_SMD:R_0603_1608Metric
- removed J10, J11, J12, J13, J14, J15, J16, J17, J9: Conn_Coaxial, Connector_Coaxial:SMA_Amphenol_132289_EdgeMount
- removed R13, R14, R15: 10k, Resistor_SMD:R_0603_1608Metric
- removed R2: 0, Resistor_SMD:R_0603_1608Metric
- removed R3, R4, R5, R6, R7, R8, R9: 22.1k, Resistor_SMD:R_0603_1608Metric
- removed U3, U4, U6: ADAR1000ACCZN, adar1000:CC-88-1_ADI
- added C62: 0.1uF, Resistor_SMD:R_0603_1608Metric, F.Cu at (303.4, 34.1)
- added C63: 10pF, Resistor_SMD:R_0603_1608Metric, F.Cu at (303.4, 36.6)
- added C64: 0.1uF, Resistor_SMD:R_0603_1608Metric, F.Cu at (303.4, 39.1)
- added C65: 10pF, Resistor_SMD:R_0603_1608Metric, F.Cu at (303.4, 41.6)
- added R16: 0, Resistor_SMD:R_0603_1608Metric, F.Cu at (303.4, 44.1)
- added R17: 10k, Resistor_SMD:R_0603_1608Metric, F.Cu at (307.4, 34.1)
- added R18: 10k, Resistor_SMD:R_0603_1608Metric, F.Cu at (307.4, 36.6)
- added R19: 0, Resistor_SMD:R_0603_1608Metric, F.Cu at (307.4, 39.1)
- added R20: 0, Resistor_SMD:R_0603_1608Metric, F.Cu at (307.4, 41.6)
- added R21: 10k, Resistor_SMD:R_0603_1608Metric, F.Cu at (307.4, 44.1)
- added R22: 0, Resistor_SMD:R_0603_1608Metric, F.Cu at (311.4, 34.1)
- added R23: 10k, Resistor_SMD:R_0603_1608Metric, F.Cu at (311.4, 36.6)
- added R24: 10k, Resistor_SMD:R_0603_1608Metric, F.Cu at (311.4, 39.1)
- added R25: 0, Resistor_SMD:R_0603_1608Metric, F.Cu at (311.4, 41.6)
- added U5: SN74AVC4T245PW, Package_SO:TSSOP-16_4.4x5mm_P0.65mm, F.Cu at (306.1, 48.7)
- moved J18 342.1 mm to (273.4, 60.2)
- moved J19 342.1 mm to (280.6, 60.2)
- moved J8 257.2 mm to (381.7, 84.6)
- moved J2 257.2 mm to (305.4, 84.5)
- moved J3 257.2 mm to (292.7, 84.5)
- moved J4 257.2 mm to (330.8, 84.5)
- moved J5 257.2 mm to (318.1, 84.5)
- moved J6 257.2 mm to (356.3, 84.6)
- moved J7 257.2 mm to (343.5, 84.5)
- moved C22 103.4 mm to (132.2, 129.9)
- moved C48 103.4 mm to (126.6, 125.2)
- moved C16 103.4 mm to (129.1, 129.9)
- moved C18 103.4 mm to (128.9, 125.5)
- moved C20 103.4 mm to (130.5, 125.5)
- moved C47 103.4 mm to (126.6, 126.7)
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Connections:
- U1 pad M3: ADAR_CS_STAGE1_1V8 -> /CSB
- U1 pad M6: ADAR_SCLK_1V8 -> /SCLK
- U2 pad A7: TX2 -> /TX1/PLL_IN
Routing:
- net GND: track 89.1 -> 0.00 mm, vias 1030 -> 0
- net TX3: track 78.5 -> 0.00 mm
- net TX2: track 78.5 -> 0.00 mm
- net TX4: track 77.7 -> 0.00 mm
- net TX1: track 77.7 -> 0.00 mm
- net OUT15: track 32.5 -> 0.00 mm
- net OUT14: track 32.5 -> 0.00 mm
- net OUT11: track 32.5 -> 0.00 mm
- net OUT7: track 32.5 -> 0.00 mm
- net OUT3: track 32.5 -> 0.00 mm
- net OUT2: track 32.4 -> 0.00 mm
- net OUT6: track 32.4 -> 0.00 mm
- net OUT10: track 32.4 -> 0.00 mm
- net +3.3V: track 32.3 -> 0.00 mm, vias 5 -> 0
- net OUT16: track 32.2 -> 0.00 mm
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- removed copper zone on F.Cu, net GND
