File: SBSP Control Board/Wilkinson Split Board/wilkinson/_autosave-trace_pretty.kicad_sch (KiCad schematic)
At the start: 85 parts, among them IC1 SN74AVC2T245RSWR, J1 Conn_01x02_Socket, J10 Conn_Coaxial, J11 Conn_Coaxial, J12 Conn_Coaxial, J13 Conn_Coaxial, J14 Conn_Coaxial, J15 Conn_Coaxial, J16 Conn_Coaxial, J17 Conn_Coaxial, J2 Conn_01x02_Socket, J3 Conn_01x20_Socket, J4 Conn_01x20_Socket, J5 Conn_01x12_Socket, J6 Conn_01x02_Pin, J7 Conn_01x02_Pin, J8 Conn_01x02_Pin, J9 Conn_Coaxial, U1 ADAR1000ACCZN, U2 SN74AVC4T245PW, U3 SN74AVC4T245PW, U4 ADAR1000ACCZN

Commit message: finished schematic and routing rev1
Other:
- note added: "going to need to go in and check all the power nets. +3.3VDC = AVDD/AVDD3 -5VDC = AVDD2 -3.3VDC = AVDD1"
Changed lines of the file:
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@@
+		)
+	)
+	(text "going to need to go in and check all the power nets.\n\n+3.3VDC = AVDD/AVDD3\n\n-5VDC = AVDD2\n\n-3.3VDC = AVDD1"
+		(exclude_from_sim no)
+		(at 319.024 192.786 0)
+		(effects
+			(font
+				(size 1.27 1.27)
+			)
 		)
 	)
