File: SBSP Control Board/Wilkinson Split Board/wilkinson/trace_pretty.kicad_sch (KiCad schematic)
At the start: 85 parts, among them IC1 SN74AVC2T245RSWR, J1 Conn_01x02_Socket, J10 Conn_Coaxial, J11 Conn_Coaxial, J12 Conn_Coaxial, J13 Conn_Coaxial, J14 Conn_Coaxial, J15 Conn_Coaxial, J16 Conn_Coaxial, J17 Conn_Coaxial, J2 Conn_01x02_Socket, J3 Conn_01x20_Socket, J4 Conn_01x20_Socket, J5 Conn_01x12_Socket, J6 Conn_01x02_Pin, J7 Conn_01x02_Pin, J8 Conn_01x02_Pin, J9 Conn_Coaxial, U1 ADAR1000ACCZN, U2 SN74AVC4T245PW, U3 SN74AVC4T245PW, U4 ADAR1000ACCZN

Commit message: redid entire layout for support
Connections:
- net +3V3 is gone; now on net +3.3V: C12.2, C13.2, C17.2, C18.2, C31.2, C32.2, IC1.7 (VCCA), R9.2, U2.1 (VCCA), U3.1 (VCCA), U3.2 (1DIR), U3.3 (2DIR)
